File: SoilMoistureMan.brd (EAGLE design)
At the start: 23.5 x 89.4 mm, 21 parts, among them Q1 BC847CSMD, Q2 BC857C, Q3 BC847CSMD, Q4 MMBTA13LT1

Commit message: committing latest updates
committing latest updates
Parts:
- R1: value 150k -> 100k
Routing:
- net GND: track 102.9 -> 80.1 mm, vias 18 -> 17
- net SOIL_PROBE_A: track 29.4 -> 28.2 mm, vias 3 -> 4
Changed lines of the file:
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@@
 <layer number="20" name="Dimension" color="15" fill="1" visible="yes" active="yes"/>
 <layer number="21" name="tPlace" color="7" fill="1" visible="yes" active="yes"/>
-<layer number="22" name="bPlace" color="7" fill="1" visible="no" active="yes"/>
+<layer number="22" name="bPlace" color="7" fill="1" visible="yes" active="yes"/>
 <layer number="23" name="tOrigins" color="15" fill="1" visible="yes" active="yes"/>
 <layer number="24" name="bOrigins" color="15" fill="1" visible="yes" active="yes"/>
@@
 <attribute name="VALUE" x="11.78" y="44.21125" size="1.27" layer="28" ratio="10" rot="MR180"/>
 </element>
-<element name="R1" library="resistor" package="R0603" value="150k" x="18.0975" y="42.38625" rot="MR90">
-<attribute name="OC_FARNELL" value="2331756" x="18.0975" y="42.38625" size="1.778" layer="28" rot="MR90" display="off"/>
+<element name="R1" library="resistor" package="R0603" value="100k" x="18.0975" y="42.38625" rot="MR90">
+<attribute name="OC_FARNELL" value="2331753" x="18.0975" y="42.38625" size="1.778" layer="28" rot="MR90" display="off"/>
 <attribute name="MF" value="TE CONNECTIVITY" x="18.0975" y="42.38625" size="1.778" layer="28" rot="MR90" display="off"/>
-<attribute name="MPN" value="CRGH0603J150K" x="18.0975" y="42.38625" size="1.778" layer="28" rot="MR90" display="off"/>
+<attribute name="MPN" value="CRGH0603J100K" x="18.0975" y="42.38625" size="1.778" layer="28" rot="MR90" display="off"/>
 </element>
 <element name="R2" library="resistor" package="R0603" value="1Meg" x="21.43125" y="51.1175" smashed="yes" rot="R90">
@@
 <attribute name="MPN" value="BCV27" x="20.0025" y="46.6725" size="1.778" layer="28" rot="MR0" display="off"/>
 </element>
-<element name="Q3" library="transistor-npn" package="SOT23" value="BC847CSMD" x="7.46125" y="46.99" rot="MR0">
+<element name="Q3" library="transistor-npn" package="SOT23" value="BC847CSMD" x="7.46125" y="46.99" smashed="yes" rot="MR0">
 <attribute name="MPN" value="BC847C-7-F" x="7.46125" y="46.99" size="1.778" layer="28" rot="MR0" display="off"/>
 <attribute name="MF" value="DIODES INC." x="7.46125" y="46.99" size="1.778" layer="28" rot="MR0" display="off"/>
 <attribute name="OC_FARNELL" value="1773609" x="7.46125" y="46.99" size="1.778" layer="28" rot="MR0" display="off"/>
+<attribute name="NAME" x="9.36625" y="48.895" size="1.27" layer="26" rot="MR0"/>
 </element>
 <element name="LED1" library="P-LCC-2_Shorter" package="P-LCC-2" value="GREEN LED" x="17.145" y="70.00875" smashed="yes" rot="R270">
@@
 <wire x1="23.1775" y1="41.28375" x2="23.01625" y2="41.445" width="0.3048" layer="16"/>
 <via x="21.43125" y="39.21125" extent="1-16" drill="0.6"/>
-<wire x1="21.43125" y1="39.21125" x2="21.43125" y2="34.6075" width="1.27" layer="1"/>
+<wire x1="21.43125" y1="39.21125" x2="21.43125" y2="35.2425" width="1.27" layer="1"/>
 <wire x1="21.43125" y1="34.6075" x2="21.11375" y2="33.81375" width="0.8128" layer="1"/>
 <wire x1="21.11375" y1="33.81375" x2="20.79625" y2="33.81375" width="0.8128" layer="1"/>
@@
 <via x="21.43125" y="35.2425" extent="1-16" drill="2.2"/>
 <via x="21.43125" y="-4.60375" extent="1-16" drill="2.2"/>
-<wire x1="21.43125" y1="35.2425" x2="21.43125" y2="27.6225" width="3.81" layer="1"/>
-<wire x1="21.43125" y1="35.2425" x2="21.43125" y2="27.78125" width="4.064" layer="16"/>
+<wire x1="21.43125" y1="34.6075" x2="21.43125" y2="27.6225" width="3.81" layer="1"/>
 <wire x1="23.1775" y1="39.84625" x2="22.5425" y2="39.21125" width="0.3048" layer="16"/>
 <wire x1="22.5425" y1="39.21125" x2="21.43125" y2="39.21125" width="0.3048" layer="16"/>
-<wire x1="21.43125" y1="35.2425" x2="21.43125" y2="34.6075" width="0" layer="19" extent="1-1"/>
-<wire x1="21.43125" y1="-4.60375" x2="21.43125" y2="27.6225" width="0" layer="19" extent="1-1"/>
+<via x="21.43125" y="28.2575" extent="1-16" drill="2.2"/>
+<wire x1="21.43125" y1="35.2425" x2="21.43125" y2="28.2575" width="3.81" layer="16"/>
+<wire x1="21.43125" y1="34.6075" x2="21.43125" y2="35.2425" width="3.81" layer="1"/>
 </signal>
 <signal name="N$3">
@@
 <wire x1="7.60875" y1="41.445" x2="7.62" y2="41.43375" width="0.3048" layer="16"/>
 <via x="7.62" y="41.43375" extent="1-16" drill="0.6"/>
-<wire x1="7.62" y1="41.43375" x2="5.3975" y2="41.43375" width="0.3048" layer="1"/>
-<wire x1="5.3975" y1="41.43375" x2="3.4925" y2="43.33875" width="0.3048" layer="1"/>
-<wire x1="6.19125" y1="50.2675" x2="4.23" y2="50.2675" width="0.3048" layer="1"/>
-<wire x1="4.23" y1="50.2675" x2="3.4925" y2="49.53" width="0.3048" layer="1"/>
-<wire x1="3.4925" y1="43.33875" x2="3.4925" y2="49.53" width="0.3048" layer="1"/>
+<wire x1="7.62" y1="41.43375" x2="5.55625" y2="41.43375" width="0.3048" layer="1"/>
+<wire x1="5.55625" y1="41.43375" x2="3.65125" y2="43.33875" width="0.3048" layer="1"/>
+<wire x1="6.19125" y1="50.2675" x2="4.38875" y2="50.2675" width="0.3048" layer="1"/>
+<wire x1="4.38875" y1="50.2675" x2="3.65125" y2="49.53" width="0.3048" layer="1"/>
+<wire x1="3.65125" y1="43.33875" x2="3.65125" y2="49.53" width="0.3048" layer="1"/>
 </signal>
 <signal name="GND">
@@
 <vertex x="29.68625" y="31.27375"/>
 <vertex x="-0.9525" y="30.95625"/>
-<vertex x="0" y="35.40125"/>
-<vertex x="-0.79375" y="35.56"/>
+<vertex x="-0.9525" y="35.71875"/>
 </polygon>
 <contactref element="BAT1" pad="-"/>
@@
 <wire x1="6.19125" y1="35.56" x2="6.50875" y2="35.2425" width="0.8128" layer="1"/>
 <via x="3.96875" y="37.465" extent="1-16" drill="0.6"/>
-<wire x1="6.50875" y1="35.2425" x2="8.89" y2="31.59125" width="0.8128" layer="1"/>
-<wire x1="3.96875" y1="37.465" x2="6.19125" y2="34.76625" width="0.8128" layer="16"/>
-<wire x1="6.19125" y1="34.76625" x2="6.985" y2="33.9725" width="0.8128" layer="16"/>
-<wire x1="6.985" y1="33.9725" x2="9.36625" y2="33.9725" width="0.8128" layer="16"/>
-<wire x1="9.36625" y1="33.9725" x2="8.5725" y2="33.17875" width="0.8128" layer="16"/>
 <wire x1="11.58875" y1="43.33875" x2="10.63625" y2="42.38625" width="0.8128" layer="1"/>
 <wire x1="10.63625" y1="42.38625" x2="10.63625" y2="39.21125" width="0.8128" layer="1"/>
@@
 <via x="19.3675" y="75.40625" extent="1-16" drill="0.6"/>
 <via x="9.2075" y="37.465" extent="1-16" drill="0.6"/>
-<via x="18.0975" y="37.465" extent="1-16" drill="0.6"/>
 <polygon width="0.6096" layer="1" isolate="0.3048">
 <vertex x="1.11125" y="31.27375"/>
@@
 <wire x1="6.50875" y1="43.97375" x2="6.50875" y2="45.8875" width="0.3048" layer="16"/>
 <wire x1="6.50875" y1="45.8875" x2="6.51125" y2="45.89" width="0.3048" layer="16"/>
-<wire x1="6.50875" y1="35.2425" x2="6.35" y2="33.9725" width="0.4064" layer="16"/>
-<wire x1="6.50875" y1="35.2425" x2="6.50875" y2="23.8125" width="2.54" layer="16"/>
-<wire x1="6.50875" y1="35.2425" x2="6.50875" y2="23.65375" width="2.54" layer="1"/>
 <via x="23.495" y="68.2625" extent="1-16" drill="0.6"/>
 <via x="4.28625" y="68.10375" extent="1-16" drill="0.6"/>
 <via x="6.50875" y="28.2575" extent="1-16" drill="2.2"/>
-<via x="21.43125" y="28.2575" extent="1-16" drill="2.2"/>
-<wire x1="18.0975" y1="37.465" x2="21.43125" y2="28.2575" width="0" layer="19" extent="1-1"/>
+<wire x1="6.50875" y1="28.2575" x2="6.50875" y2="35.2425" width="3.81" layer="16"/>
+<wire x1="6.50875" y1="35.2425" x2="6.50875" y2="28.2575" width="3.81" layer="1"/>
+<via x="18.0975" y="37.465" extent="1-16" drill="0.6"/>
 </signal>
 <signal name="N$10">
@@
 <wire x1="10.31875" y1="45.4025" x2="12.22375" y2="47.3075" width="0.3048" layer="1"/>
 <wire x1="12.22375" y1="47.3075" x2="12.22375" y2="50.2675" width="0.3048" layer="1"/>
-<wire x1="21.2725" y1="48.26" x2="19.52625" y2="50.00625" width="0.3048" layer="16"/>
+<wire x1="21.2725" y1="48.41875" x2="19.52625" y2="50.00625" width="0.3048" layer="16"/>
 <wire x1="19.52625" y1="50.00625" x2="17.93875" y2="50.00625" width="0.3048" layer="16"/>
 <wire x1="17.93875" y1="50.00625" x2="16.98625" y2="49.05375" width="0.3048" layer="16"/>
@@
 <wire x1="10.63625" y1="49.68875" x2="10.63625" y2="48.41875" width="0.3048" layer="1"/>
 <contactref element="Q4" pad="B"/>
-<wire x1="21.2725" y1="48.26" x2="21.2725" y2="47.14875" width="0.3048" layer="16"/>
+<wire x1="21.2725" y1="48.41875" x2="21.2725" y2="47.14875" width="0.3048" layer="16"/>
 <wire x1="21.2725" y1="47.14875" x2="20.955" y2="46.83125" width="0.3048" layer="16"/>
 <wire x1="20.955" y1="46.83125" x2="20.955" y2="45.575" width="0.3048" layer="16"/>
@@
 <signal name="N$5">
 <contactref element="R7" pad="1"/>
-<wire x1="18.7325" y1="67.78625" x2="17.62125" y2="66.675" width="0.6096" layer="1"/>
-<wire x1="17.62125" y1="66.675" x2="18.57375" y2="65.7225" width="0.6096" layer="1"/>
-<wire x1="18.57375" y1="65.7225" x2="17.145" y2="64.29375" width="0.6096" layer="1"/>
-<wire x1="17.145" y1="64.29375" x2="19.05" y2="62.38875" width="0.6096" layer="1"/>
+<wire x1="18.7325" y1="67.78625" x2="17.62125" y2="66.675" width="0.8636" layer="1"/>
+<wire x1="17.62125" y1="66.675" x2="18.57375" y2="65.7225" width="0.8128" layer="1"/>
+<wire x1="18.57375" y1="65.7225" x2="17.145" y2="64.29375" width="0.762" layer="1"/>
+<wire x1="17.145" y1="64.29375" x2="19.05" y2="62.38875" width="0.7112" layer="1"/>
 <via x="19.05" y="62.38875" extent="1-16" drill="0.6"/>
 <wire x1="18.25625" y1="51.9675" x2="18.25625" y2="52.07" width="0.3048" layer="1"/>
@@
 <contactref element="LED1" pad="A"/>
 <contactref element="LED2" pad="A"/>
-<wire x1="18.7325" y1="67.78625" x2="18.7325" y2="70.00125" width="0.6096" layer="1"/>
+<wire x1="18.7325" y1="67.78625" x2="18.7325" y2="70.00125" width="0.9652" layer="1"/>
 <wire x1="18.7325" y1="70.00125" x2="18.725" y2="70.00875" width="0.6096" layer="1"/>
 <wire x1="9.525" y1="73.18375" x2="17.78" y2="73.18375" width="0.4064" layer="16"/>
@@
 <contactref element="Q3" pad="3"/>
 <wire x1="7.46125" y1="48.10125" x2="5.3975" y2="48.10125" width="0.3048" layer="16"/>
-<wire x1="7.46125" y1="48.10125" x2="7.46125" y2="48.09" width="0" layer="19" extent="16-16"/>
+<wire x1="7.46125" y1="48.09" x2="7.46125" y2="48.10125" width="0.4064" layer="16"/>
 </signal>
 <signal name="N$1">
