File: SoilMoistureMan.sch (EAGLE design)
At the start: 20 parts, among them Q1 BC847CSMD, Q2 BC857C, Q3 BC847CSMD, Q4 MMBTA13LT1

Commit message: Committing latest updates on CAD C
Committing latest updates on CAD C
Parts:
- LED1, LED2: value GENERIC_0603_SMD_LED -> GREEN LED; device led:LEDSML0603 -> P-LCC-2_Shorter:LEDP-LCC-2; MF AVAGO TECHNOLOGIES -> OSRAM; MPN ASMT-CR00 -> LGT67K-H2K1-24-Z; OC_FARNELL 1863233 -> 1226376
- R7: value 2k -> 560R; MF TE CONNECTIVITY / NEOHM -> TE CONNECTIVITY; MPN CPF0603F2K0C1 -> CRGH0603J560R; OC_FARNELL 1527506 -> 2331724
- VR1: device adafruit:TRIMPOTTC33X -> P-LCC-2_Shorter:TRIMPOTTC33X
Other:
- note added: "Change R3, R1, R7 values. consider using a FET to switch the LED on. due to the 0.65v min at the cathode of the LED"
- note added: "SOME CONTAMINATION OF THE SOIL WILL OCCUR. DO NOT USE WITH EDIBLE PLANTS."
- note removed: "SOME CONTAMINATION OF THE SOIL WILL OCCUR. DO NOT USE ON EDIBLE PLANTS."
Changed lines of the file:
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@@
 </classes>
 <parts>
-<part name="Q3" library="transistor-npn" deviceset="BC847*" device="SMD" technology="C">
-<attribute name="MF" value="DIODES INC."/>
-<attribute name="MPN" value="BC847C-7-F"/>
-<attribute name="OC_FARNELL" value="1773609"/>
-</part>
 <part name="SUPPLY2" library="supply2" deviceset="GND" device=""/>
 <part name="Q1" library="transistor-npn" deviceset="BC847*" device="SMD" technology="C">
@@
 </part>
 <part name="SUPPLY1" library="supply2" deviceset="GND" device=""/>
-<part name="VR1" library="adafruit" deviceset="TRIMPOT" device="TC33X" value="100k">
+<part name="VR1" library="P-LCC-2_Shorter" deviceset="TRIMPOT" device="TC33X" value="100k">
 <attribute name="MF" value="VISHAY SFERNICE"/>
 <attribute name="MPN" value="TS53YJ104MR10"/>
@@
 <attribute name="OC_FARNELL" value="2141628"/>
 </part>
-<part name="R7" library="resistor" deviceset="R-EU_" device="R0603" value="2k">
-<attribute name="MF" value="TE CONNECTIVITY / NEOHM"/>
-<attribute name="MPN" value="CPF0603F2K0C1"/>
-<attribute name="OC_FARNELL" value="1527506"/>
+<part name="R7" library="resistor" deviceset="R-EU_" device="R0603" value="560R">
+<attribute name="MF" value="TE CONNECTIVITY"/>
+<attribute name="MPN" value="CRGH0603J560R"/>
+<attribute name="OC_FARNELL" value="2331724"/>
 </part>
 <part name="C1" library="resistor" deviceset="C-EU" device="C0603" value="1uF">
@@
 <attribute name="OC_FARNELL" value="1759016"/>
 </part>
-<part name="LED1" library="led" deviceset="LED" device="SML0603" value="GENERIC_0603_SMD_LED">
-<attribute name="MF" value="AVAGO TECHNOLOGIES"/>
-<attribute name="MPN" value="ASMT-CR00"/>
-<attribute name="OC_FARNELL" value="1863233"/>
-</part>
 <part name="F1" library="rcl" deviceset="R-EU_" device="R0805" value="100MA PTC FUSE">
 <attribute name="MF" value="BOURNS"/>
@@
 <attribute name="MPN" value="PMEG3010EJ,115"/>
 <attribute name="OC_FARNELL" value="1757770"/>
-</part>
-<part name="LED2" library="led" deviceset="LED" device="SML0603" value="GENERIC_0603_SMD_LED">
-<attribute name="MF" value="AVAGO TECHNOLOGIES"/>
-<attribute name="MPN" value="ASMT-CR00"/>
-<attribute name="OC_FARNELL" value="1863233"/>
 </part>
 <part name="R8" library="resistor" deviceset="R-EU_" device="R0603" value="0R0">
@@
 <attribute name="OC_FARNELL" value="9846689"/>
 </part>
+<part name="Q3" library="transistor-npn" deviceset="BC847*" device="SMD" technology="C">
+<attribute name="MF" value="DIODES INC."/>
+<attribute name="MPN" value="BC847C-7-F"/>
+<attribute name="OC_FARNELL" value="1773609"/>
+</part>
+<part name="LED1" library="P-LCC-2_Shorter" deviceset="LED" device="P-LCC-2" value="GREEN LED">
+<attribute name="MF" value="OSRAM"/>
+<attribute name="MPN" value="LGT67K-H2K1-24-Z"/>
+<attribute name="OC_FARNELL" value="1226376"/>
+</part>
+<part name="LED2" library="P-LCC-2_Shorter" deviceset="LED" device="P-LCC-2" value="GREEN LED">
+<attribute name="MF" value="OSRAM"/>
+<attribute name="MPN" value="LGT67K-H2K1-24-Z"/>
+<attribute name="OC_FARNELL" value="1226376"/>
+</part>
 </parts>
 <sheets>
@@
 <plain>
 <text x="-27.94" y="15.24" size="1.778" layer="91">&lt;- TO THE SOIL</text>
-<text x="-45.72" y="-10.16" size="1.778" layer="91">SOME CONTAMINATION OF THE SOIL WILL OCCUR. DO NOT USE ON EDIBLE PLANTS. </text>
+<text x="-45.72" y="-10.16" size="1.778" layer="91">SOME CONTAMINATION OF THE SOIL WILL OCCUR. DO NOT USE WITH EDIBLE PLANTS. </text>
 <text x="-58.42" y="-7.62" size="1.778" layer="91">WARNING: THIS PROJECT WILL CAUSE ELECTROLYSIS AND SO THE PLATING ON THE LEGS WILL DEGRADE OVER TIME. </text>
+<text x="-27.94" y="101.6" size="1.778" layer="91">Change R3, R1, R7 values. consider using a FET to switch the LED on. due to the 0.65v min at the cathode of the LED</text>
 </plain>
 <instances>
-<instance part="Q3" gate="G$1" x="68.58" y="43.18" rot="MR0">
-<attribute name="OC_FARNELL" x="68.58" y="43.18" size="1.778" layer="96" display="off"/>
-<attribute name="MF" x="68.58" y="43.18" size="1.778" layer="96" display="off"/>
-<attribute name="MPN" x="68.58" y="43.18" size="1.778" layer="96" display="off"/>
-</instance>
 <instance part="SUPPLY2" gate="GND" x="-35.56" y="53.34"/>
 <instance part="Q1" gate="G$1" x="17.78" y="22.86">
@@
 <attribute name="MPN" x="106.68" y="60.96" size="1.778" layer="96" display="off"/>
 </instance>
-<instance part="LED1" gate="G$1" x="116.84" y="71.12">
-<attribute name="OC_FARNELL" x="116.84" y="71.12" size="1.778" layer="96" display="off"/>
-<attribute name="MF" x="116.84" y="71.12" size="1.778" layer="96" display="off"/>
-<attribute name="MPN" x="116.84" y="71.12" size="1.778" layer="96" display="off"/>
-</instance>
 <instance part="F1" gate="G$1" x="-38.1" y="91.44">
 <attribute name="OC_FARNELL" x="-38.1" y="91.44" size="1.778" layer="96" display="off"/>
@@
 <attribute name="MF" x="-17.78" y="76.2" size="1.778" layer="96" rot="R90" display="off"/>
 <attribute name="MPN" x="-17.78" y="76.2" size="1.778" layer="96" rot="R90" display="off"/>
-</instance>
-<instance part="LED2" gate="G$1" x="127" y="71.12">
-<attribute name="OC_FARNELL" x="127" y="71.12" size="1.778" layer="96" display="off"/>
-<attribute name="MF" x="127" y="71.12" size="1.778" layer="96" display="off"/>
-<attribute name="MPN" x="127" y="71.12" size="1.778" layer="96" display="off"/>
 </instance>
 <instance part="R8" gate="G$1" x="66.04" y="68.58" rot="R90">
@@
 <attribute name="MF" x="111.76" y="43.18" size="1.778" layer="96" display="off"/>
 <attribute name="MPN" x="111.76" y="43.18" size="1.778" layer="96" display="off"/>
-<attribute name="NAME" x="105.41" y="50.8" size="1.778" layer="95"/>
+<attribute name="NAME" x="110.49" y="48.26" size="1.778" layer="95"/>
+</instance>
+<instance part="Q3" gate="G$1" x="68.58" y="43.18" rot="MR0">
+<attribute name="OC_FARNELL" x="68.58" y="43.18" size="1.778" layer="96" rot="MR0" display="off"/>
+<attribute name="MF" x="68.58" y="43.18" size="1.778" layer="96" rot="MR0" display="off"/>
+<attribute name="MPN" x="68.58" y="43.18" size="1.778" layer="96" rot="MR0" display="off"/>
+</instance>
+<instance part="LED1" gate="G$1" x="116.84" y="71.12">
+<attribute name="OC_FARNELL" x="116.84" y="71.12" size="1.778" layer="96" display="off"/>
+<attribute name="MF" x="116.84" y="71.12" size="1.778" layer="96" display="off"/>
+<attribute name="MPN" x="116.84" y="71.12" size="1.778" layer="96" display="off"/>
+</instance>
+<instance part="LED2" gate="G$1" x="127" y="71.12">
+<attribute name="OC_FARNELL" x="127" y="71.12" size="1.778" layer="96" display="off"/>
+<attribute name="MF" x="127" y="71.12" size="1.778" layer="96" display="off"/>
+<attribute name="MPN" x="127" y="71.12" size="1.778" layer="96" display="off"/>
 </instance>
 </instances>
@@
 <net name="GND" class="0">
 <segment>
-<pinref part="Q3" gate="G$1" pin="E"/>
 <wire x1="66.04" y1="38.1" x2="66.04" y2="33.02" width="0.1524" layer="91"/>
 <wire x1="66.04" y1="33.02" x2="91.44" y2="33.02" width="0.1524" layer="91"/>
@@
 <junction x="91.44" y="33.02"/>
 <pinref part="Q4" gate="G$1" pin="E"/>
+<pinref part="Q3" gate="G$1" pin="E"/>
 </segment>
 <segment>
@@
 <wire x1="99.06" y1="78.74" x2="99.06" y2="60.96" width="0.1524" layer="91"/>
 <wire x1="99.06" y1="60.96" x2="104.14" y2="60.96" width="0.1524" layer="91"/>
-<pinref part="Q3" gate="G$1" pin="B"/>
 <wire x1="71.12" y1="43.18" x2="83.82" y2="43.18" width="0.1524" layer="91"/>
 <wire x1="83.82" y1="43.18" x2="99.06" y2="60.96" width="0.1524" layer="91"/>
@@
 <pinref part="R6" gate="G$1" pin="1"/>
 <pinref part="C2" gate="G$1" pin="1"/>
+<pinref part="Q3" gate="G$1" pin="B"/>
 </segment>
 </net>
@@
 <wire x1="116.84" y1="66.04" x2="116.84" y2="63.5" width="0.1524" layer="91"/>
 <pinref part="C2" gate="G$1" pin="2"/>
-<pinref part="LED1" gate="G$1" pin="C"/>
-<pinref part="LED2" gate="G$1" pin="C"/>
 <wire x1="116.84" y1="63.5" x2="116.84" y2="60.96" width="0.1524" layer="91"/>
 <wire x1="127" y1="66.04" x2="127" y2="63.5" width="0.1524" layer="91"/>
@@
 <wire x1="116.84" y1="45.72" x2="116.84" y2="60.96" width="0.1524" layer="91"/>
 <junction x="116.84" y="60.96"/>
+<pinref part="LED1" gate="G$1" pin="C"/>
+<pinref part="LED2" gate="G$1" pin="C"/>
 </segment>
 </net>
@@
 <wire x1="116.84" y1="73.66" x2="116.84" y2="76.2" width="0.1524" layer="91"/>
 <pinref part="R7" gate="G$1" pin="1"/>
-<pinref part="LED1" gate="G$1" pin="A"/>
 <wire x1="116.84" y1="76.2" x2="116.84" y2="78.74" width="0.1524" layer="91"/>
 <wire x1="116.84" y1="76.2" x2="127" y2="76.2" width="0.1524" layer="91"/>
 <junction x="116.84" y="76.2"/>
+<wire x1="127" y1="76.2" x2="127" y2="73.66" width="0.1524" layer="91"/>
+<pinref part="LED1" gate="G$1" pin="A"/>
 <pinref part="LED2" gate="G$1" pin="A"/>
-<wire x1="127" y1="76.2" x2="127" y2="73.66" width="0.1524" layer="91"/>
 </segment>
 </net>
 <net name="N$7" class="0">
 <segment>
-<pinref part="Q3" gate="G$1" pin="C"/>
 <wire x1="66.04" y1="63.5" x2="66.04" y2="60.96" width="0.1524" layer="91"/>
 <pinref part="R8" gate="G$1" pin="1"/>
@@
 <wire x1="71.12" y1="60.96" x2="66.04" y2="60.96" width="0.1524" layer="91"/>
 <junction x="66.04" y="60.96"/>
-</segment>
-</net>
+<pinref part="Q3" gate="G$1" pin="C"/>
+</segment>
+</net>

Commit message: committing latest updates
committing latest updates
Parts:
- R1: value 150k -> 100k; MPN CRGH0603J150K -> CRGH0603J100K; OC_FARNELL 2331756 -> 2331753
Changed lines of the file:
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@@
 <attribute name="OC_FARNELL" value="1216354"/>
 </part>
-<part name="R1" library="resistor" deviceset="R-EU_" device="R0603" value="150k">
+<part name="R1" library="resistor" deviceset="R-EU_" device="R0603" value="100k">
 <attribute name="MF" value="TE CONNECTIVITY"/>
-<attribute name="MPN" value="CRGH0603J150K"/>
-<attribute name="OC_FARNELL" value="2331756"/>
+<attribute name="MPN" value="CRGH0603J100K"/>
+<attribute name="OC_FARNELL" value="2331753"/>
 </part>
 <part name="R2" library="resistor" deviceset="R-EU_" device="R0603" value="1Meg">
